File: charge_control.kicad_sch (KiCad schematic)
At the start: 0 parts

Commit message: Prepared STS1_BATT_TEST.
Other:
- note added: "Choose a MOSFET that enables or disables the charging of the battery. You most likely want to choose a PFET here. I probably won't need cooling, as the charging currents won't exceed 2A by much."
Changed lines of the file:
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@@
 	(generator_version "8.0")
 	(paper "A4")
+	(text "Choose a MOSFET that enables or disables the charging \nof the battery. You most likely want to choose a PFET here.\nI probably won't need cooling, as the charging currents won't\nexceed 2A by much."
+		(exclude_from_sim no)
+		(at 69.342 37.846 0)
+		(effects
+			(font
+				(size 1.27 1.27)
+			)
+		)
+	)
 	(hierarchical_label "SOURCE"
 		(shape input)
