File: shunt.kicad_sch (KiCad schematic)
At the start: 0 parts

Commit message: Prepared STS1_BATT_TEST.
Other:
- note added: "Choose a suitable shunt resistor here. Note that the load MOSFET's resistance is ~5 mOhm. Depending on the shunts resistance, it will be subjected to more or less power dissipation. It will have to withstand this power dissipation. It may even need an extra heat sink. It's totally fine if you choose a through hole component here."
Changed lines of the file:
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@@
 	(generator_version "8.0")
 	(paper "A4")
+	(text "Choose a suitable shunt resistor here.\nNote that the load MOSFET's resistance is ~5 mOhm. \nDepending on the shunts resistance, it will be subjected to\nmore or less power dissipation. It will have to withstand this \npower dissipation. It may even need an extra heat sink. It's totally\nfine if you choose a through hole component here."
+		(exclude_from_sim no)
+		(at 17.78 32.512 0)
+		(effects
+			(font
+				(size 1.27 1.27)
+			)
+			(justify left)
+		)
+	)
 	(hierarchical_label "LOW"
 		(shape input)
